File: ArduinoNanoDcLoad.kicad_pcb (KiCad board)
At the start: 2 copper layers, 35 parts, among them P1 DCLOAD+, P2 DCLOAD-, P3 CONN_01X15, P4 CONN_01X15, Q1 IRFP250N, U1 LMC6484

Commit message: * updated
Parts:
- added C7: 100n, Capacitors_ThroughHole:C_Rect_L4_W2.5_P2.5, F.Cu at (125.7, 43.2)
- added D2: 5,1V, Diodes_ThroughHole:Diode_DO-35_SOD27_Horizontal_RM10, F.Cu at (125.7, 61.0)
- C2: footprint Capacitors_ThroughHole:C_Radial_D10_L20_P5 -> Capacitors_ThroughHole:C_Rect_L4_W2.5_P2.5
- R14: value 10 -> 1
- R17: value 1 -> 10
- R5: value 1 -> 470
- R6: value 470 -> 1k
- R7: value 1k -> 1
- moved C5 136.5 mm to (166.4, 50.8)
- moved R3 117.8 mm to (110.5, 116.8), turned to 270 degrees
- moved R18 113.7 mm to (163.8, 111.8)
- moved D1 108.8 mm to (158.8, 116.8)
- moved C6 101.2 mm to (163.8, 104.1)
- moved R14 99.6 mm to (87.6, 58.4)
- moved R19 98.6 mm to (153.7, 127.0)
- moved R4 96.9 mm to (115.6, 132.1), turned to 90 degrees
- moved R17 90.4 mm to (133.3, 94.0), turned to 270 degrees
- moved C4 90.0 mm to (128.3, 127.0), turned to 90 degrees
- moved P4 78.3 mm to (179.1, 63.5)
- moved R6 71.2 mm to (156.2, 63.5), turned to 270 degrees
- moved C1 71.1 mm to (143.5, 119.4), turned to 180 degrees
- moved R1 70.3 mm to (143.5, 109.2)
- moved C2 69.2 mm to (146.1, 45.7)
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Connections:
- P3 pad 1: /TX/PD1 -> (no net)
- P3 pad 10: /AIN1/PD7 -> (no net)
- P3 pad 11: /CLKO/PB0 -> (no net)
- P3 pad 13: /OC1B/PB2 -> (no net)
- P3 pad 14: /MISO/PB4 -> (no net)
- P3 pad 15: /MOSI/OC2/PB3 -> (no net)
- P3 pad 2: /RX/PD0 -> (no net)
- P3 pad 5: /INT0/PD2 -> (no net)
- P3 pad 6: /INT1/PD3 -> (no net)
- P3 pad 7: /T0/PD4 -> (no net)
- P3 pad 8: /T1/PD5 -> (no net)
- P3 pad 9: /AIN0/PD6 -> (no net)
- P4 pad 1: /VIN -> (no net)
- P4 pad 10: /ADC2/PC2 -> (no net)
- P4 pad 11: /ADC1/PC1 -> (no net)
- P4 pad 12: /ADC0/PC0 -> (no net)
- P4 pad 13: /AREF -> (no net)
- P4 pad 14: /3V3 -> (no net)
- P4 pad 15: /SCK/PB5 -> (no net)
- P4 pad 4: /5V -> (no net)
- P4 pad 7: /ADC5/PC5/SCL -> (no net)
- P4 pad 8: /ADC4/SDA/PC4 -> (no net)
- P4 pad 9: /ADC3/PC3 -> (no net)
- R14 pad 1: Net-(C4-Pad2) -> Net-(Q1-Pad3)
- R17 pad 1: Net-(Q1-Pad3) -> Net-(C4-Pad2)
- R21 pad 1: Net-(R21-Pad1) -> /ADC6
- R22 pad 2: Net-(R21-Pad1) -> /ADC6
- R5 pad 1: Net-(Q1-Pad3) -> Net-(Q1-Pad1)
- R5 pad 2: GND -> Net-(C3-Pad1)
- R6 pad 1: Net-(Q1-Pad1) -> Net-(Q1-Pad3)
- R6 pad 2: Net-(C3-Pad1) -> Net-(C3-Pad2)
- R7 pad 2: Net-(C3-Pad2) -> GND
- U1 pad 4: +12V -> (no net)
- U1 pad 8: Net-(R21-Pad1) -> /ADC6
Routing:
- net GND: track 90.3 -> 0.00 mm
- net (no net): track 25.4 -> 0.00 mm
Other:
- board outline added: 200 x 100 mm

Commit message: * updated pcb layout
Parts:
- added C11: 100n, Capacitors_ThroughHole:C_Rect_L4_W2.5_P2.5, F.Cu at (163.8, 127.0)
- added C8: 220µ, Capacitors_ThroughHole:C_Radial_D10_L20_P5, F.Cu at (161.3, 58.4)
- added C9: 100n, Capacitors_ThroughHole:C_Rect_L4_W2.5_P2.5, F.Cu at (158.8, 124.5)
- added CON1: BARREL_JACK, Connect:JACK_ALIM, F.Cu at (156.2, 40.6)
- added DS1: LCD16X2, Display:WC1602A, F.Cu at (222.2, 61.0)
- added R23: 2k, Resistors_ThroughHole:Resistor_Horizontal_RM15mm, F.Cu at (138.4, 50.8)
- added R24: 680, Resistors_ThroughHole:Resistor_Horizontal_RM15mm, F.Cu at (181.6, 94.0)
- added R25: 470, Resistors_ThroughHole:Resistor_Horizontal_RM15mm, F.Cu at (186.7, 109.2)
- added RV1: 10k, Potentiometers:Potentiometer_Trimmer-Piher-PT15-h5_vertical, F.Cu at (176.5, 116.8)
- added RV2: 200, Potentiometers:Potentiometer_Trimmer-Piher-PT15-h5_vertical, F.Cu at (135.9, 43.2)
- added U2: LM7812, TO_SOT_Packages_THT:TO-220_Neutral123_Vertical, F.Cu at (146.1, 53.3)
- added U3: LM317T, TO_SOT_Packages_THT:TO-220_Neutral123_Vertical, F.Cu at (130.8, 58.4)
- moved R18 23.4 mm to (148.6, 94.0)
- moved P4 23.0 mm to (181.6, 40.6)
- moved P3 23.0 mm to (168.9, 40.6)
- moved R19 20.5 mm to (143.5, 109.2)
- moved C2 20.3 mm to (146.1, 66.0), turned to 270 degrees
- moved C5 19.8 mm to (153.7, 66.0), turned to 180 degrees
- moved D1 18.0 mm to (156.2, 99.1)
- moved R22 12.7 mm to (123.2, 58.4)
- moved C6 11.5 mm to (165.1, 92.7)
- moved R6 11.4 mm to (151.1, 73.7)
- moved R5 11.4 mm to (115.6, 109.2), turned to 90 degrees
- moved R17 8.03 mm to (125.7, 96.5)
- moved C7 7.62 mm to (118.1, 43.2)
- moved D2 7.62 mm to (118.1, 61.0)
- moved C4 7.18 mm to (133.3, 121.9), turned to 270 degrees
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Connections:
- P3 pad 10: (no net) -> /AIN1/PD7
- P3 pad 11: (no net) -> /CLKO/PB0
- P3 pad 12: /OC1A/PB1 -> (no net)
- P3 pad 13: (no net) -> /OC1B/PB2
- P3 pad 7: (no net) -> /T0/PD4
- P3 pad 8: (no net) -> /T1/PD5
- P3 pad 9: (no net) -> /AIN0/PD6
- P4 pad 4: (no net) -> +5V
- R1 pad 2: /OC1A/PB1 -> (no net)
- R21 pad 1: /ADC6 -> Net-(R21-Pad1)
- R22 pad 2: /ADC6 -> Net-(R21-Pad1)
- U1 pad 4: (no net) -> +12V
- U1 pad 8: /ADC6 -> Net-(R21-Pad1)

Commit message: * update
Parts:
- moved R24 84.1 mm to (108.0, 53.3), turned to 90 degrees
- moved C9 80.7 mm to (141.0, 45.7), turned to 0 degrees
- moved C7 74.1 mm to (191.8, 50.8), turned to 90 degrees
- moved C5 73.7 mm to (102.9, 119.4), turned to 270 degrees
- moved C6 47.1 mm to (186.7, 50.8), turned to 90 degrees
- moved R17 42.3 mm to (102.9, 132.1), turned to 0 degrees
- moved C4 38.4 mm to (95.2, 127.0)
- moved R18 35.9 mm to (184.2, 88.9)
- moved R19 35.9 mm to (179.1, 104.1)
- moved R23 26.2 mm to (115.6, 38.1)
- moved R25 20.5 mm to (184.2, 129.5)
- moved R3 18.9 mm to (125.7, 102.9)
- moved R22 18.5 mm to (118.1, 76.2)
- moved R20 17.8 mm to (108.0, 76.2)
- moved R21 17.8 mm to (113.0, 61.0)
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Connections:
- U1 pad 10: Net-(Q1-Pad3) -> (no net)
- U1 pad 12: (no net) -> Net-(Q1-Pad3)
- U1 pad 13: (no net) -> Net-(R20-Pad1)
- U1 pad 14: (no net) -> Net-(R21-Pad1)
- U1 pad 8: Net-(R21-Pad1) -> (no net)
- U1 pad 9: Net-(R20-Pad1) -> (no net)

Commit message: update
Other:
- net class Default removed
- net class HeavyLoadNet removed
