File: ArduinoNanoDcLoad.kicad_sch (KiCad schematic)
At the start: 49 parts, among them CON1 BARREL_JACK, P1 DCLOAD+, P2 DCLOAD-, P3 CONN_01X15, P4 CONN_01X15, Q1 IRFP250N, U1 LMC6484, U2 LM7812, U3 LM317T

Commit message: update
Parts:
- C4: value 10µ -> 10µ/50V; Field4 (none) -> ECAP6.3x5.5-2.2mm
Changed lines of the file:
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@@
       (effects (font (size 1.27 1.27)) (justify left))
     )
-    (property "Value" "10µ" (id 1) (at 122.555 39.37 0)
+    (property "Value" "10µ/50V" (id 1) (at 118.11 40.005 0)
       (effects (font (size 1.27 1.27)) (justify left))
     )
@@
     )
     (property "Datasheet" "" (id 3) (at 121.92 36.83 0))
+    (property "Field4" "ECAP6.3x5.5-2.2mm" (id 4) (at 121.92 36.83 0)
+      (effects (font (size 1.27 1.27)) hide)
+    )
     (pin "1")
     (pin "2")
@@
     )
     (path "/00000000-0000-0000-0000-000058389373"
-      (reference "C4") (unit 1) (value "10µ") (footprint "Capacitors_ThroughHole:C_Radial_D10_L20_P5")
+      (reference "C4") (unit 1) (value "10µ/50V") (footprint "Capacitors_ThroughHole:C_Radial_D10_L20_P5")
     )
     (path "/00000000-0000-0000-0000-0000583892dc"
